Commit message: feat: add basic Gazebo simulation and robot spawn

File: ros2_ws/src/ci_bot_description/urdf/ci_bot.urdf.xacro (robot description, xacro)
@@ -17,4 +17,13 @@
     <color rgba="0.45 0.45 0.45 1.0"/>
   </material>
+  <!-- =============================================================== -->
+  <!-- Inertial-free root frame for KDL / robot_state_publisher -->
+  <!-- =============================================================== -->
+  <link name="base_footprint"/>
+  <joint name="base_footprint_joint" type="fixed">
+    <parent link="base_footprint"/>
+    <child link="base_link"/>
+    <origin xyz="0 0 0" rpy="0 0 0"/>
+  </joint>
   <!-- =============================================================== -->
   <!-- Main chassis -->
